File: soc_power.kicad_sch (KiCad schematic)
At the start: 63 parts, among them Q10 MMBT3904, Q2 MMBT3904, Q3 MMBT3904, U2 Allwinner_V3S, U3 TMI7003x

Commit message: Add V3s variant with smaller exposed GND pad
Parts:
- U2: footprint Package_QFP_Allwinner:LQFP-128_14x14mm_P0.4mm_EPAD_8x8mm -> Package_QFP_Allwinner:LQFP-128_14x14mm_P0.4mm_EPAD_5.72x5.72mm
Changed lines of the file:
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@@
       (effects (font (size 1.27 1.27)) (justify right))
     )
-    (property "Footprint" "Package_QFP_Allwinner:LQFP-128_14x14mm_P0.4mm_EPAD_8x8mm" (at 191.77 36.83 0)
+    (property "Footprint" "Package_QFP_Allwinner:LQFP-128_14x14mm_P0.4mm_EPAD_5.72x5.72mm" (at 191.77 36.83 0)
       (effects (font (size 1.27 1.27)) hide)
     )
@@
       (effects (font (size 1.27 1.27)) (justify left))
     )
-    (property "Footprint" "Package_QFP_Allwinner:LQFP-128_14x14mm_P0.4mm_EPAD_8x8mm" (at 186.69 6.35 0)
+    (property "Footprint" "Package_QFP_Allwinner:LQFP-128_14x14mm_P0.4mm_EPAD_5.72x5.72mm" (at 186.69 6.35 0)
       (effects (font (size 1.27 1.27)) hide)
     )
@@
       (effects (font (size 1.27 1.27)) (justify left))
     )
-    (property "Footprint" "Package_QFP_Allwinner:LQFP-128_14x14mm_P0.4mm_EPAD_8x8mm" (at 176.53 67.31 0)
-      (effects (font (size 1.27 1.27)) hide)
-    )
+    (property "Footprint" "Package_QFP_Allwinner:LQFP-128_14x14mm_P0.4mm_EPAD_5.72x5.72mm" (at 176.53 67.31 0)
+      (effects (font (size 1.27 1.27)) hide)
+    )

Commit message: Fix LCSC part numbers
Parts:
- R22: LCSC C25768 -> C25741
- U2: LCSC (none) -> C2687449
Changed lines of the file:
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@@
       (effects (font (size 1.27 1.27)) hide)
     )
-    (property "LCSC" "C25768" (at 95.25 120.65 0)
+    (property "LCSC" "C25741" (at 95.25 120.65 0)
       (effects (font (size 1.27 1.27)) hide)
     )
@@
     )
     (property "Datasheet" "" (at 191.77 36.83 0)
+      (effects (font (size 1.27 1.27)) hide)
+    )
+    (property "LCSC" "C2687449" (at 161.29 64.77 0)
       (effects (font (size 1.27 1.27)) hide)
     )
@@
       (effects (font (size 1.27 1.27)) hide)
     )
+    (property "LCSC" "C2687449" (at 156.21 34.29 0)
+      (effects (font (size 1.27 1.27)) hide)
+    )
     (pin "110")
     (pin "111")
@@
       (effects (font (size 1.27 1.27)) hide)
     )
+    (property "LCSC" "C2687449" (at 146.05 95.25 0)
+      (effects (font (size 1.27 1.27)) hide)
+    )
