File: soc_spi_nor.kicad_sch (KiCad schematic)
At the start: 6 parts, among them U2 Allwinner_V3S, U5 W25Q128JVS

Commit message: Add V3s variant with smaller exposed GND pad
Parts:
- U2: footprint Package_QFP_Allwinner:LQFP-128_14x14mm_P0.4mm_EPAD_8x8mm -> Package_QFP_Allwinner:LQFP-128_14x14mm_P0.4mm_EPAD_5.72x5.72mm
Changed lines of the file:
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@@
       (effects (font (size 1.27 1.27)))
     )
-    (property "Footprint" "Package_QFP_Allwinner:LQFP-128_14x14mm_P0.4mm_EPAD_8x8mm" (at 82.55 72.39 0)
+    (property "Footprint" "Package_QFP_Allwinner:LQFP-128_14x14mm_P0.4mm_EPAD_5.72x5.72mm" (at 82.55 72.39 0)
       (effects (font (size 1.27 1.27)) hide)
     )

Commit message: Fix LCSC part numbers
Parts:
- U2: LCSC (none) -> C2687449
- U5: LCSC (none) -> C97521
Changed lines of the file:
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@@
+      (effects (font (size 1.27 1.27)) hide)
+    )
+    (property "LCSC" "C2687449" (at 54.61 41.91 0)
       (effects (font (size 1.27 1.27)) hide)
     )
@@
       (effects (font (size 1.27 1.27)) hide)
     )
+    (property "LCSC" "C97521" (at 102.87 50.8 0)
+      (effects (font (size 1.27 1.27)) hide)
+    )
