File: soc_unused.kicad_sch (KiCad schematic)
At the start: 3 parts, among them U2 Allwinner_V3S

Commit message: Add V3s variant with smaller exposed GND pad
Parts:
- U2: footprint Package_QFP_Allwinner:LQFP-128_14x14mm_P0.4mm_EPAD_8x8mm -> Package_QFP_Allwinner:LQFP-128_14x14mm_P0.4mm_EPAD_5.72x5.72mm
Changed lines of the file:
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@@
       (effects (font (size 1.27 1.27)))
     )
-    (property "Footprint" "Package_QFP_Allwinner:LQFP-128_14x14mm_P0.4mm_EPAD_8x8mm" (at 156.21 124.46 0)
+    (property "Footprint" "Package_QFP_Allwinner:LQFP-128_14x14mm_P0.4mm_EPAD_5.72x5.72mm" (at 156.21 124.46 0)
       (effects (font (size 1.27 1.27)) hide)
     )
@@
       (effects (font (size 1.27 1.27)))
     )
-    (property "Footprint" "Package_QFP_Allwinner:LQFP-128_14x14mm_P0.4mm_EPAD_8x8mm" (at 154.94 86.36 0)
-      (effects (font (size 1.27 1.27)) hide)
-    )
+    (property "Footprint" "Package_QFP_Allwinner:LQFP-128_14x14mm_P0.4mm_EPAD_5.72x5.72mm" (at 154.94 86.36 0)
+      (effects (font (size 1.27 1.27)) hide)
+    )

Commit message: Fix LCSC part numbers
Parts:
- U2: LCSC (none) -> C2687449
Changed lines of the file:
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@@
+      (effects (font (size 1.27 1.27)) hide)
+    )
+    (property "LCSC" "C2687449" (at 128.27 93.98 0)
       (effects (font (size 1.27 1.27)) hide)
     )
@@
       (effects (font (size 1.27 1.27)) hide)
     )
+    (property "LCSC" "C2687449" (at 127 55.88 0)
+      (effects (font (size 1.27 1.27)) hide)
+    )
